File: 8 Pin DIN to 9 Pin Mini DIN.kicad_pcb (KiCad board)
At the start: 2 copper layers, 15.8 x 36.2 mm, 6 parts, among them J1 DIN-8, J2 MD-90SM

Commit message: new and improved
Parts:
- moved J2 4.20 mm to (198.6, 127.0)
- moved REF** 4.20 mm to (205.2, 118.0)
- moved REF** 1.40 mm to (192.0, 104.6)
Routing:
- net GND: track 5.29 -> 55.0 mm, vias 7 -> 8
- net LEFT: track 14.6 -> 13.2 mm
- net 5V: track 21.3 -> 19.9 mm
- net BLUE: track 22.7 -> 21.3 mm
- net SYNC: track 19.9 -> 18.6 mm
- net RIGHT: track 8.53 -> 7.28 mm
- net GREEN: track 26.2 -> 25.6 mm
- net RED: track 25.2 -> 24.7 mm
Other:
- board size 15.8 x 36.2 mm -> 16.8 x 40.4 mm
- board text added: "Tinkerplunk.com PC Engine/TurboDuo to HDRetrovision Adapter 2.0"
- board text removed: "Tinkerplunk.com PC Engine/TurboDuo to HDRetrovision Adapter"
